File: BreadBoard Power Supply/BreadBoard Power Supply.kicad_sch (KiCad schematic)
At the start: 0 parts

Commit message: Schematic work
Parts:
- added C1, C2, C3, C4, C6: 10uF, Capacitor_SMD:C_1206_3216Metric_Pad1.33x1.80mm_HandSolder, symbol Device:C
- added C10, C11, C7, C8: 22uF, Capacitor_SMD:C_1206_3216Metric_Pad1.33x1.80mm_HandSolder, symbol Device:C
- added C5: 1uF, Capacitor_SMD:C_1206_3216Metric_Pad1.33x1.80mm_HandSolder, symbol Device:C
- added C9: 100nF, Capacitor_SMD:C_1206_3216Metric_Pad1.33x1.80mm_HandSolder, symbol Device:C
- added D1, D2: RB550VAM-30TR, BreadBoard Power Supply:DIO_RB160VAM_ROM-L, symbol Device:D
- added D3: APT3216QBC/D, BreadBoard Power Supply:LED_APT3216QBC_D, symbol Device:LED
- added D4: APT3216CGCK, BreadBoard Power Supply:LED_APT3216QBC_D, symbol Device:LED
- added F1: 0ZCG0150BF2C, BreadBoard Power Supply:0ZCG_BEL, symbol Device:Polyfuse
- added H1, H2: MountingHole, symbol Mechanical:MountingHole
- added J1, J2, J3, J4: 22285051, Connector_PinSocket_2.54mm:PinSocket_1x05_P2.54mm_Vertical, symbol Connector:Conn_01x05_Pin
- added J5: 2171750001, BreadBoard Power Supply:2171750001_MOL, symbol bbps:2171750001
- added L1: .47uH, BreadBoard Power Supply:IND_LQH32PNR47NN0L, symbol Device:L
- added L2, L3: 4.7uH, BreadBoard Power Supply:IND_NRS4012T100MDGJV_TAY, symbol Device:L
- added R1, R2, R5, R8, R9: 5.1k, Resistor_SMD:R_1206_3216Metric_Pad1.30x1.75mm_HandSolder, symbol Device:R_US
- added R3, R6: 100k, Resistor_SMD:R_1206_3216Metric_Pad1.30x1.75mm_HandSolder, symbol Device:R_US
- added R4, R7: 20k, Resistor_SMD:R_1206_3216Metric_Pad1.30x1.75mm_HandSolder, symbol Device:R_US
- added U1: TPS6285021HQDRLRQ1, BreadBoard Power Supply:DRL0008A-MFG, symbol bbps:TPS6285021HQDRLRQ1
- added U2: BD81870EFV-ME2, BreadBoard Power Supply:HTSSOP-B20_ROM-L, symbol bbps:BD81870EFV-ME2
- added U3: GPI-152-3013, BreadBoard Power Supply:SW_GPI-152-3013_CWI, symbol bbps:GPI-152-3013
Connections:
- new net: R3.1, R4.2, U2.8 (NON1)
- new net: D2.2 (A), L3.2, U2.15 (LX2)
- new net: L3.1, U2.14 (HS2L)
- new net: D3.1 (K), R5.1
- new net: C10.2, C11.1
- new net: C1.2, C2.2, F1.2, U1.1 (VIN), U1.2 (EN), U1.3 (MODE)
- new net: L1.1, U1.7 (SW)
- new net: J5.B5 (CC2), R2.1
- new net: C9.2, R4.1, U2.7 (VREF)
- new net: D4.2 (A), R8.1
- new net: R7.2, R9.1, U2.20 (INV2)
- new net: J5.A5 (CC1), R1.2
- new net: D1.1 (K), L2.2, U2.10 (LX1)
- new net: C7.2, C8.1
- new net: R6.1, R9.2
- new net +3.3V: C3.2, C4.2, C5.2, C6.2, L1.2, U1.5 (FB), U2.1 (VDDA), U2.11 (VDDP), U2.12 (VDDP), U2.13 (VDDP), U2.2 (STB2), U2.3 (STB1), U2.4 (SEQON)
- new net +5V: C10.1, D2.1 (K), J1.1 (Pin_1), J1.2 (Pin_2), J1.3 (Pin_3), J1.4 (Pin_4), J1.5 (Pin_5), R6.2, R8.2, U2.17 (VOUT2)
- new net -5V: C7.1, D1.2 (A), J2.1 (Pin_1), J2.2 (Pin_2), J2.3 (Pin_3), J2.4 (Pin_4), J2.5 (Pin_5), R3.2, R5.2
- new net GND: C1.1, C11.2, C2.1, C3.1, C4.1, C5.1, C6.1, C8.2, C9.1, D3.2 (A), D4.1 (K), J3.1 (Pin_1), J3.2 (Pin_2), J3.3 (Pin_3), J3.4 (Pin_4), J3.5 (Pin_5), J4.1 (Pin_1), J4.2 (Pin_2), J4.3 (Pin_3), J4.4 (Pin_4), J4.5 (Pin_5), J5.A12 (GND_2), J5.B12 (GND), L2.1, R1.1, R2.2, R7.1, U1.4 (COMP_FSET), U1.6 (PG), U1.8 (GND), U2.16 (GNDP), U2.18 (DIS2), U2.19 (GNDA), U2.9 (DIS1), U2.EPAD, U3.10, U3.7, U3.8, U3.9
- new net SWITCHED_VOLTAGE: F1.1, U3.4, U3.5
- new net USB_VOLTAGE: J5.A9 (VBUS_2), J5.B9 (VBUS), U3.2, U3.3
- no-connect marks 0 -> 3
Other:
- note added: "-5V = - (100k/20k) x 1.0V"
- note added: "3.3V -> +5V and -5V"
- note added: "5.004V = (((100k + 5.1k) + 20k)/20k) x 0.8V Using 5.1k for BOM reduction"
- note added: "Blue (-5V)"
- note added: "Green (+5V)"
- note added: "On/Off Switch"
- note added: "USB 5V -> 3.3V"
- note added: "USB-C"

Commit message: PCB work
Parts:
- removed J1, J2, J3, J4: 22285051, Connector_PinSocket_2.54mm:PinSocket_1x05_P2.54mm_Vertical, symbol Connector:Conn_01x05_Pin
- added C12, C13: 1uF, Capacitor_SMD:C_1206_3216Metric_Pad1.33x1.80mm_HandSolder, symbol Device:C
- added J2, J3: Conn_02x05_Top_Bottom, Connector_PinSocket_2.54mm:PinSocket_2x05_P2.54mm_Vertical, symbol Connector_Generic:Conn_02x05_Top_Bottom
- H1, H2: footprint (none) -> BreadBoard Power Supply:RubberFoot
- renumbered C9 to C1, C3 to C10, C4 to C11, C7 to C2, C8 to C3, C5 to C4, C6 to C5, C10 to C6, C11 to C7, C1 to C8, C2 to C9, J5 to J1, L2 to L1, L3 to L2, L1 to L3, R4 to R3, R3 to R4, R7 to R5, R9 to R6, R6 to R7, R5 to R8, R8 to R9, U3 to U1, U1 to U3
Connections:
- net +5V: now also C12.2, J2.1 (Pin_1), J2.3 (Pin_3), J2.5 (Pin_5), J2.7 (Pin_7), J2.9 (Pin_9)
- net -5V: now also C13.2, J2.10 (Pin_10), J2.2 (Pin_2), J2.4 (Pin_4), J2.6 (Pin_6), J2.8 (Pin_8)
- net GND: now also C1.2, C12.1, C13.1, J3.1 (Pin_1), J3.10 (Pin_10), J3.2 (Pin_2), J3.3 (Pin_3), J3.4 (Pin_4), J3.5 (Pin_5), J3.6 (Pin_6), J3.7 (Pin_7), J3.8 (Pin_8), J3.9 (Pin_9); no longer C1.1
- net SWITCHED_VOLTAGE: now also U1.3; no longer U1.5
- net USB_VOLTAGE: now also U1.5; no longer U1.3
- net at R3.1, U2.7 (VREF): now also C1.1; no longer C1.2
Other:
- moved on the sheet: C1
