File: BreadBoard Power Supply/BreadBoard Power Supply.kicad_pcb (KiCad board)
At the start: 2 copper layers, 8.6 x 4.4 mm, 36 parts, among them J1 Conn_01x05_Pin, J2 Conn_01x05_Pin, J3 Conn_01x05_Pin, J4 Conn_01x05_Pin, J5 2171750001, U1 TPS6285021HQDRLRQ1, U2 BD81870EFV-ME2, U3 GPI-152-3013

Commit message: PCB work
Parts:
- removed the J1 at (91.6, 65.4)
- removed J4: Conn_01x05_Pin, Connector_PinSocket_2.54mm:PinSocket_1x05_P2.54mm_Vertical
- added C12: 1uF, Capacitor_SMD:C_1206_3216Metric_Pad1.33x1.80mm_HandSolder, F.Cu at (80.8, 26.9)
- added C13: 1uF, Capacitor_SMD:C_1206_3216Metric_Pad1.33x1.80mm_HandSolder, F.Cu at (80.7, 30.2)
- added H1: MountingHole, BreadBoard Power Supply:RubberFoot, B.Cu at (53.7, 37.0)
- added H2: MountingHole, BreadBoard Power Supply:RubberFoot, B.Cu at (53.5, 61.4)
- C1: renamed from C9; value .1uF -> 100nF
- D1, D2: value D -> RB550VAM-30TR
- D3: value LED -> APT3216QBC/D
- D4: value LED -> APT3216CGCK
- F1: value Polyfuse -> 0ZCG0150BF2C
- J2, J3: value Conn_01x05_Pin -> Conn_02x05_Top_Bottom; footprint Connector_PinSocket_2.54mm:PinSocket_1x05_P2.54mm_Vertical -> Connector_PinSocket_2.54mm:PinSocket_2x05_P2.54mm_Vertical
- moved J1 65.4 mm to (25.1, 34.3), turned to -90 degrees
- moved R1 51.6 mm to (36.5, 31.4), turned to 180 degrees
- moved R2 50.8 mm to (36.6, 37.5)
- moved F1 49.7 mm to (48.0, 67.1)
- moved C3 46.2 mm to (52.3, 44.4), turned to 180 degrees
- moved C8 43.8 mm to (57.1, 70.7), turned to 90 degrees
- moved C2 38.9 mm to (59.4, 44.4), turned to 180 degrees
- moved J2 38.3 mm to (93.7, 27.3), turned to 90 degrees
- moved U2 38.2 mm to (76.9, 49.8)
- moved C9 37.9 mm to (62.0, 70.7), turned to 90 degrees
- moved C1 32.8 mm to (66.2, 44.7), turned to -90 degrees
- moved R9 32.5 mm to (91.5, 23.6), turned to 180 degrees
- moved L1 31.9 mm to (74.3, 57.2), turned to 90 degrees
- moved U1 28.2 mm to (29.2, 55.3)
- moved U3 27.7 mm to (68.0, 65.8)
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- renumbered C3 to C10, C4 to C11, C7 to C2, C8 to C3, C5 to C4, C6 to C5, C10 to C6, C11 to C7, C1 to C8, C2 to C9, J5 to J1, L2 to L1, L3 to L2, L1 to L3, R4 to R3, R3 to R4, R7 to R5, R9 to R6, R6 to R7, R5 to R8, R8 to R9, U3 to U1, U1 to U3
Connections:
- J2 pad 1: -5V -> +5V
- J2 pad 3: -5V -> +5V
- J2 pad 5: -5V -> +5V
- U1 pad 3: USB_VOLTAGE -> SWITCHED_VOLTAGE
- U1 pad 5: SWITCHED_VOLTAGE -> USB_VOLTAGE
Routing:
- net Net-(U2-VREF): track 0.00 -> 14.4 mm
- net Net-(U2-INV2): track 0.00 -> 14.0 mm
- net Net-(U2-NON1): track 0.00 -> 12.4 mm
- net Net-(J1-CC2): track 0.00 -> 8.04 mm
- net Net-(J1-CC1): track 0.00 -> 7.73 mm
- net Net-(R6-Pad2): track 0.00 -> 5.46 mm
- net +3.3V: track 0.00 -> 4.58 mm, vias 0 -> 8
- net Net-(C2-Pad2): track 0.00 -> 3.96 mm
- net Net-(D3-K): track 0.00 -> 3.84 mm
- net Net-(D4-A): track 0.00 -> 3.72 mm
- net GND: track 0.00 -> 3.56 mm, vias 0 -> 2
- net Net-(U3-SW): track 0.00 -> 2.89 mm
- net Net-(C6-Pad2): track 0.00 -> 2.87 mm
- net Net-(D2-A): track 0.00 -> 1.26 mm
- net +5V: track 0.00 -> 0.56 mm, vias 0 -> 8
- added copper zone on B.Cu, net +3.3V
- added copper zone on F.Cu, net +3.3V
- added copper zone on B.Cu, net +5V
- added copper zone on F.Cu, net +5V
- added copper zone on F.Cu, net -5V
- added copper zone on B.Cu, net GND
- added copper zone on F.Cu, net GND
- added copper zone on F.Cu, net Net-(D1-K)
- added copper zone on F.Cu, net Net-(D2-A)
- added copper zone on F.Cu, net Net-(U2-HS2L)
- added copper zone on F.Cu, net Net-(U3-EN)
- added copper zone on F.Cu, net Net-(U3-SW)
- added copper zone on F.Cu, net SWITCHED_VOLTAGE
- added copper zone on F.Cu, net USB_VOLTAGE
Other:
- board size 8.6 x 4.4 mm -> 85 x 57 mm
- board text added: "2171750001"
- board text added: "PTC - 1812"
- board text added: "USB-C"

Commit message: Pushing Proto 1 Files
Parts:
- removed the C10 at (72.6, 69.8)
- removed the C9 at (62.0, 70.7)
- removed U3: TPS6285021HQDRLRQ1, BreadBoard Power Supply:DRL0008A-MFG
- added C12: 1uF, Capacitor_SMD:C_1206_3216Metric_Pad1.33x1.80mm_HandSolder, F.Cu at (65.8, 60.7)
- added C13: 22uF, Capacitor_SMD:C_1206_3216Metric_Pad1.33x1.80mm_HandSolder, F.Cu at (81.2, 70.5)
- added C14: 22uF, Capacitor_SMD:C_1206_3216Metric_Pad1.33x1.80mm_HandSolder, F.Cu at (85.6, 70.5)
- added D5: APT3216CGCK, BreadBoard Power Supply:LED_APT3216QBC_D, F.Cu at (100.8, 65.5)
- added G***: LOGO, BreadBoard Power Supply:vt_logo, F.Cu at (71.8, 34.4)
- added G***: LOGO, BreadBoard Power Supply:logo, F.Cu at (44.9, 52.2)
- added G***: LOGO, BreadBoard Power Supply:BOM, B.Cu at (81.2, 50.0)
- added R10: 5.1k, Resistor_SMD:R_1206_3216Metric_Pad1.30x1.75mm_HandSolder, F.Cu at (94.5, 65.5)
- added U1: L6982N33DR, BreadBoard Power Supply:SOIC127P600X175-8N, F.Cu at (64.2, 67.5)
- C11: value 10uF -> 100nF
- J1: footprint BreadBoard Power Supply:2171750001_MOL -> BreadBoard Power Supply:2171750001
- L3: value .47uH -> 22uH; footprint BreadBoard Power Supply:IND_LQH32PNR47NN0L -> BreadBoard Power Supply:IND_PCC-M0748M-LE_PAN-L
- moved C11 13.8 mm to (64.2, 74.3), turned to 180 degrees
- moved L3 4.48 mm to (72.5, 69.3), turned to 90 degrees
- moved F1 2.10 mm to (45.9, 67.1)
- moved U1 1.30 mm to (29.5, 56.5)
- moved C2 0.11 mm to (66.3, 44.6), turned to 90 degrees
- renumbered C13 to C1, C12 to C10, C1 to C2, C2 to C3, C3 to C4, C4 to C5, C5 to C6, C8 to C7, C6 to C8, C7 to C9, H2 to H1, H1 to H2
Connections:
- C11 pad 1: GND -> Net-(IC1-SW)
- C11 pad 2: +3.3V -> Net-(IC1-BOOT)
- C2 pad 1: GND -> Net-(U2-VREF)
- C2 pad 2: Net-(U2-VREF) -> GND
- J3 pad 1: GND -> +3.3V
- J3 pad 3: GND -> +3.3V
- J3 pad 5: GND -> +3.3V
- J3 pad 7: GND -> +3.3V
- J3 pad 9: GND -> +3.3V
- L3 pad 1: Net-(U3-SW) -> Net-(IC1-SW)
Routing:
- net Net-(IC1-BOOT): track 0.00 -> 8.31 mm
- net Net-(IC1-VCC): track 0.00 -> 7.99 mm
- net +3.3V: track 4.58 -> 0.00 mm
- net Net-(D5-A): track 0.00 -> 2.94 mm
- net Net-(U3-SW): track 2.89 -> 0.00 mm
- net Net-(IC1-EN/CLKIN(~{)}): track 0.00 -> 2.07 mm
- net GND: track 3.56 -> 2.20 mm, vias 2 -> 1
- net +5V: track 0.56 -> 0.00 mm
- added copper zone on F.Cu, net Net-(IC1-SW)
- removed copper zone on F.Cu, net Net-(U3-SW)
Other:
- board text added: "*"
- board text added: "100K"
- board text added: "100nF"
- board text added: "10uF"
- board text added: "1uF"
- board text added: "20K"
- board text added: "22uF"
- board text added: "22uH"
- board text added: "4.7uH"
- board text added: "5.1K"
- board text added: "AMP LAB Intermediate Soldering Certification Board"
- board text added: "BD81870EFV-ME2"
- board text added: "BLUE"
- board text added: "BREADBOARD +5V,-5V, AND +3.3V POWER SUPPLY"
- board text added: "Breadboard Goes Here"
- board text added: "Designed By: Shane Wyman"
- board text added: "Dot"
- board text added: "GREEN"
- board text added: "Goes Here"
- board text added: "Here"
- board text added: "JLCJLCJLCJLC"
- board text added: "L6982N33DR"
- board text added: "LAB"
- board text added: "Notch Goes"
- board text added: "The AMP"
- board text added: "amp-lab.org"
