File: BreadBoard Power Supply/BreadBoard Power Supply-backups/BreadBoard Power Supply-2025-10-06_155314/BreadBoard Power Supply.kicad_sch (KiCad schematic)
At the start: 41 parts, among them IC1 L6982N33DR, J1 2171750001, J2 Conn_02x05_Top_Bottom, J3 Conn_02x05_Top_Bottom, U1 GPI-152-3013, U2 BD81870EFV-ME2

Commit message: Pushing Proto 1 Files
Parts:
- removed C12: 1uF, Capacitor_SMD:C_1206_3216Metric_Pad1.33x1.80mm_HandSolder, symbol Device:C
- removed C13, C14: 22uF, Capacitor_SMD:C_1206_3216Metric_Pad1.33x1.80mm_HandSolder, symbol Device:C
- removed D5: APT3216CGCK, BreadBoard Power Supply:LED_APT3216QBC_D, symbol Device:LED
- removed IC1: L6982N33DR, BreadBoard Power Supply:SOIC127P600X175-8N, symbol bbps:L6982N33DR
- removed R10: 5.1k, Resistor_SMD:R_1206_3216Metric_Pad1.30x1.75mm_HandSolder, symbol Device:R_US
- added C10, C9: 10uF, Capacitor_SMD:C_1206_3216Metric_Pad1.33x1.80mm_HandSolder, symbol Device:C
- added U3: TPS6285021HQDRLRQ1, BreadBoard Power Supply:DRL0008A-MFG, symbol bbps:TPS6285021HQDRLRQ1
- C11: value 100nF -> 10uF
- J1: footprint BreadBoard Power Supply:2171750001 -> BreadBoard Power Supply:2171750001_MOL
- L3: value 22uH -> .47uH; footprint BreadBoard Power Supply:IND_PCC-M0748M-LE_PAN-L -> BreadBoard Power Supply:IND_LQH32PNR47NN0L
- renumbered C2 to C1, C10 to C12, C1 to C13, C3 to C2, C4 to C3, C5 to C4, C6 to C5, C8 to C6, C9 to C7, C7 to C8, H2 to H1, H1 to H2
Connections:
- net +3.3V: now also C11.2, C10.2, U3.5 (FB)
- net GND: now also C11.1, C10.1, C9.1, U3.4 (COMP_FSET), U3.6 (PG), U3.8 (GND); no longer J1.MH1, J1.MH2, J1.MH3, J1.MH4
- net at C8.2, F1.2: now also C9.2, U3.1 (VIN), U3.2 (EN), U3.3 (MODE)
- net at L3.1: now also U3.7 (SW); no longer C11.1
Other:
- note removed: "ETQ-P4M220KFM"
- note removed: "Green (+3.3V)"
- moved on the sheet: C8, F1, L3
